File: output.brd (EAGLE design)
At the start: 77.5 x 31.4 mm, 14 parts, among them Q1 FQP30N06L

Commit message: correct diode lead order in part/package name
MUR860 and RHRP3060 have pin 1 as cathode and pin 2 as anode,
so s/TO-220AC/TO-220CA/ to avoid confusion.
Parts:
- D2: device djm:TO-220ACS-HS -> djm:TO-220CAS-HS
Changed lines of the file:
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@@
 <element name="Q1" library="djm" package="TO-220BV-HS" value="FQP30N06L" x="43.18" y="13.97" rot="R270"/>
 <element name="SCR1" library="djm" package="TO-220V-HS" value="SK055R" x="31.75" y="13.97" rot="R90"/>
-<element name="D2" library="djm" package="TO-220ACS-HS" value="RHRP3060" x="11.43" y="13.97" rot="R270"/>
+<element name="D2" library="djm" package="TO-220CAS-HS" value="RHRP3060" x="11.43" y="13.97" rot="R270"/>
 <element name="JP1" library="pinhead" package="1X05" value="" x="74.93" y="13.97" smashed="yes" rot="R270">
 <attribute name="NAME" x="74.8538" y="24.2062" size="1.27" layer="25" ratio="10" rot="R270"/>
