File: photo-trigger.sch (EAGLE design)
At the start: 49 parts, among them Q1 PN2907, Q2 PN2907, Q3 20MHz, U1 ATMEGA324PA-PU

Commit message: correct device name to match library
Parts:
- VR1, VR2: value RECOMREE-0505S -> RECOM-REE-0505S; device djm:RECOMREE-0505S -> djm:RECOM-REE-0505S
Changed lines of the file:
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@@
 <part name="GND19" library="supply1" deviceset="GNDIO" device=""/>
 <part name="P+11" library="supply1" deviceset="+5V" device=""/>
-<part name="VR2" library="djm" deviceset="RECOMREE-0505S" device=""/>
+<part name="VR2" library="djm" deviceset="RECOM-REE-0505S" device=""/>
 <part name="C3" library="rcl" deviceset="C-EU" device="050-035X075" value="0.1uF"/>
 <part name="C1" library="rcl" deviceset="C-EU" device="050-035X075" value="0.1uF"/>
@@
 <part name="GND2" library="supply1" deviceset="GNDIO" device=""/>
 <part name="P+2" library="supply1" deviceset="+5V" device=""/>
-<part name="VR1" library="djm" deviceset="RECOMREE-0505S" device=""/>
+<part name="VR1" library="djm" deviceset="RECOM-REE-0505S" device=""/>
 <part name="FRAME1" library="frames" deviceset="DINA4_L" device=""/>
 <part name="FRAME2" library="frames" deviceset="DINA4_L" device=""/>

Commit message: revised after building v1.0 boards; lots of fixes
ripped out power status indicator circuit - it didn't work.
replaced with a simple power LED.

fixed footprint problem for Recom REE isolated VRMs

rewired LCD socket to be easier to handle at the LCD end

fixed MCU AREF and AGND

expanded prototype area; embiggened pads to make them easier to
solder
Parts:
- removed D1: 6.2V, diode:ZENER-DIODEDO35Z10
- removed JP5: LCD, pinhead:PINHD-2X8
- removed Q1, Q2: PN2907, djm:PN2907
- removed R4: 100K, rcl:R-EU_0207/10
- removed R5: 470, rcl:R-EU_0207/10
- added +5VI: +5VI, wirepad:1,6/0,9
- added +5VO: +5VO, wirepad:1,6/0,9
- added C8: 0.1uF, rcl:C-EU050-035X075
- added C9: 10uF, rcl:C-EU050-035X075
- added GNDI: GNDI, wirepad:1,6/0,9
- added GNDO: GNDO, wirepad:1,6/0,9
- added GNDP2: GND, wirepad:1,6/0,9
- added LCD: (no value), pinhead:PINHD-2X8
- added VCCP2: VCC, wirepad:1,6/0,9
- R1: value 100K -> 100
- VR1, VR2: value RECOM-REE-0505S -> REE-0505S
- VR3: value RECOM-R-785.0-0.5 -> R-785.0-0.5
Connections:
- removed net BATT_LOW: JP8.6, R5.1
- removed net LCD_CONTRAST: JP5.16, TRIM1.S
- removed net LCD_DB_4: JP5.7, U1.PD3
- removed net LCD_DB_5: JP5.9, U1.PD2
- removed net LCD_DB_6: JP5.11, U1.PD1
- removed net LCD_DB_7: JP5.13, U1.PD0
- removed net N$20: D1.A, R1.2, R2.1
- removed net N$21: Q1.B, R2.2
- removed net N$22: Q1.C, R3.2, R4.1
- removed net N$27: Q2.C, R5.2
- removed net N$43: Q2.B, R4.2
- new net AREF: C8.1, U1.AREF
- new net AVCC: R1.2, U1.AVCC
- new net LCD_DB4: LCD.11, U1.PD3
- new net LCD_DB5: LCD.12, U1.PD2
- new net LCD_DB6: LCD.13, U1.PD1
- new net LCD_DB7: LCD.14, U1.PD0
- new net LCD_UNU: LCD.10, LCD.7, LCD.8, LCD.9, R2.1
- new net LCD_V0: LCD.3, TRIM1.S
- net +5V: now also +5VI.P
- net GND: now also C8.2, C9.2, GNDP2.P, JP8.6, LCD.1, LCD.16, R2.2, TRIM1.E; no longer JP5.10, JP5.12, JP5.14, JP5.2, JP5.4, JP5.6, JP5.8, R1.1, TRIM1.A, U1.AREF
- net GNDI: now also GNDO.P
- net GNDIO: now also GNDI.P
- net LCD_EN: now also LCD.6; no longer JP5.1
- net LCD_RS: now also LCD.4; no longer JP5.5
- net LCD_RW: now also LCD.5; no longer JP5.3
- net VCC: now also C9.1, LCD.15, LCD.2, R1.1, R3.2, TRIM1.A, VCCP2.P; no longer JP5.15, TRIM1.E, U1.AVCC
- net VDD: now also +5VO.P
- net VIN: no longer D1.C, Q1.E, Q2.E
Other:
- moved on the sheet: C2, C4, C7, R3, VR3

Commit message: few more layout tweaks; embiggen more wirepads
Parts:
- +5VI, +5VO, GND, GNDI, GNDO, GNDP2, PA6, PA7, PC0, PC1, PC2, PC3, PC4, PC5, PC6, PC7, VCC, VCCP2: device wirepad:1,6/0,9 -> djm:PAD1.9/0.9
- LP3: value (none) -> LCD
- renumbered LCD to LP3
